File: WiFiShield.brd (EAGLE design)
At the start: 69.2 x 53.3 mm, 35 parts, among them IC3 CC3000, J4 Arduino-compatible headers, Q1 2N7002, Q2 2N7002, Q3 2N7002, Q4 2N7002, Q5 2N7002

Commit message: tweaked readme
Parts:
- removed J35, J37, J67: (no value), freetronics-master-v1:1X02
- removed R17, R18: 10kΩ, freetronics-master-v1:0603
- added C1: 10pF, freetronics-master-v1:C0402
- added C2: 2.2µF, freetronics-master-v1:0603
- added C3: 470pF, freetronics-master-v1:0603
- added IC1: MIC5219-3.3YM5, SparkFun:SOT23-5
- added J10, J5, J9: (no value), freetronics-luke:SJ
- added R11, R12: 10kΩ, freetronics-master-v1:0603
- C4: value 1µF -> 2.2µF
- C6: value 10pF -> 1µF; device freetronics-master-v1:C0402 -> freetronics-master-v1:0603
- J1, J2, J3: device freetronics-luke:SJ -> freetronics-master-v1:1X02
- J4: value Arduino-compatible headers -> (none); device Arduino-Various:NO-OUTLINE-OCTAGONAL-NOTEXT -> freetronics-luke:SJ
- J7: value (none) -> Arduino-compatible headers; device freetronics-luke:SJ -> Arduino-Various:NO-OUTLINE-OCTAGONAL-NOTEXT
- R10, R9: value 10kΩ -> 0Ω
- R3, R4: value 0Ω -> 10kΩ
- moved SY 78.8 mm to (62.9, 45.1)
- moved R9 34.4 mm to (50.8, 19.4), turned to 0 degrees
- moved J4 31.4 mm to (58.4, 47.0), turned to 90 degrees
- moved J3 29.1 mm to (66.0, 36.8), turned to 270 degrees
- moved C6 25.0 mm to (46.4, 34.6), turned to 0 degrees
- moved Q5 24.8 mm to (55.9, 42.5)
- moved J1 24.1 mm to (66.0, 24.1), turned to 270 degrees
- moved R10 22.0 mm to (46.4, 23.5), turned to 90 degrees
- moved J7 21.6 mm to (35.6, 25.4), turned to 270 degrees
- moved J2 20.5 mm to (45.7, 29.2), turned to 270 degrees
- moved Q4 17.1 mm to (38.7, 42.5)
- moved R8 17.1 mm to (41.3, 42.5), turned to 270 degrees
- moved R7 16.8 mm to (28.6, 47.6), turned to 270 degrees
- moved R4 16.2 mm to (38.7, 39.4), turned to 180 degrees
- moved R3 14.9 mm to (27.3, 39.4), turned to 180 degrees
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- renumbered IC3 to IC2, J378 to J8
Connections:
- new net N$43: C3.2, IC1.4
- net !CC3000_CS_3.3V: now also Q4.2, R4.1; no longer Q2.2, R6.1
- net !CC3000_CS_5V: now also J10.1, J9.1, Q4.3, R8.1; no longer J3.1, J7.1, Q2.3, R5.1
- net +3V3: now also C4.1, C6.2, IC1.5, R1.2, R11.2, R3.2, R4.2; no longer C4.2, R10.2, R17.2, R6.2, R8.2
- net +5V: now also C2.2, IC1.1, IC1.3, J7.5V, R12.2, R6.2, R8.2; no longer J4.5V, R1.2, R18.2, R9.2
- net 3V3: now also J7.3V3; no longer J4.3V3
- net CC3000_EN: now also J2.2; no longer J35.2
- net CC3000_IRQ_3.3V: now also Q5.2, R11.1; no longer Q4.2, R8.1
- net CC3000_IRQ_5V: now also J4.1, J5.1, Q5.3, R12.1; no longer J1.1, J2.1, Q4.3, R7.1
- net GND: now also C2.1, C3.1, C4.2, C6.1, IC1.2, J7.GND0, J7.GND1, J7.GND2; no longer C4.1, J4.GND0, J4.GND1, J4.GND2
- net MISO_3.3V: now also Q1.2, R1.1; no longer Q5.2, R10.1
- net MISO_5V: now also J7.12, Q1.3, R5.1; no longer J4.12, Q5.3, R9.1
- net MOSI_3.3V: now also Q2.2, R2.1; no longer Q3.2, R17.1
- net MOSI_5V: now also J7.11, Q2.3, R6.1; no longer J4.11, Q3.3, R18.1
- net N$1: now also R10.2; no longer R3.2
- net N$103: now also C1.1; no longer C6.1
- net N$11: now also J10.2, J7.10; no longer J4.10, J7.2
- net N$15: now also R9.2; no longer R4.2
- net N$16: now also C1.2; no longer C6.2
- net N$2: now also R10.1; no longer R3.1
- net N$4: now also J5.2, J7.3; no longer J2.2, J4.3
- net N$5: now also R9.1; no longer R4.1
- net N$6: now also J7.2; no longer J1.2
- net N$7: now also J7.9, J9.2; no longer J3.2, J4.9
- net N$9: now also J7.8; no longer J4.8
- net RES_1: now also J1.2; no longer J67.2
- net RES_2: now also J1.1; no longer J67.1
- net RES_3: now also J2.1; no longer J35.1
- net SCK_3.3V: now also Q3.2, R3.1; no longer Q1.2, R2.1
- net SCK_5V: now also J7.13, Q3.3, R7.1; no longer J4.13, Q1.3, R1.1
- net VIN: now also J7.VIN; no longer J4.VIN
- net WL_UART_RX: now also J3.1; no longer J37.1
- net WL_UART_TX: now also J3.2; no longer J37.2
Routing:
- net +5V: track 21.0 -> 110.7 mm, vias 2 -> 3
- net +3V3: track 34.0 -> 89.4 mm, vias 2 -> 6
- net RES_3: track 0.00 -> 3.92 mm
- net CC3000_EN: track 0.00 -> 3.87 mm
- net N$2: track 0.00 -> 3.49 mm
- net N$1: track 0.00 -> 3.35 mm
- net N$6: track 0.00 -> 3.05 mm
- net N$5: track 0.00 -> 3.01 mm
- net N$15: track 0.00 -> 2.88 mm
- net N$43: track 0.00 -> 1.75 mm
Other:
- board text added: "Board Fab: 0.8mm FR4, 2-layer 35µm Cu."
