File: WiFiShield.sch (EAGLE design)
At the start: 35 parts, among them IC3 CC3000, J1 SJ, J2 SJ, J3 SJ, J4 Arduino-compatible headers, J6 SJ, J7 SJ, Q1 2N7002, Q2 2N7002, Q3 2N7002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

Commit message: foo
Parts:
- removed J35, J37, J67: (no value), freetronics-master-v1:M02PTH
- removed J378: (no value), freetronics-master-v1:M03PTH
- removed R17, R18: 10kΩ, freetronics-master-v1:RESISTOR0603
- added C1: 10pF, freetronics-master-v1:CAP0402
- added C2: 2.2µF, freetronics-master-v1:CAP0603
- added C3: 470pF, freetronics-master-v1:CAP0603
- added IC1: MIC5219-3.3YM5, SparkFun:V_REG_LDOSMD
- added J10, J5, J9: SJ, freetronics-luke:SJ
- added J8: (no value), freetronics-master-v1:M03PTH
- added R11, R12: 10kΩ, freetronics-master-v1:RESISTOR0603
- C4: value 1µF -> 2.2µF
- C6: value 10pF -> 1µF; device freetronics-master-v1:CAP0402 -> freetronics-master-v1:CAP0603; PACKAGE 0402 -> 0603
- J1, J2, J3: value SJ -> (none); device freetronics-luke:SJ -> freetronics-master-v1:M02PTH
- J4: value Arduino-compatible headers -> SJ; device Arduino-Various:ARDUINO-USBNO-OUTLINE-NO-TEXT-OCTAGONAL -> freetronics-luke:SJ
- J7: value SJ -> Arduino-compatible headers; device freetronics-luke:SJ -> Arduino-Various:ARDUINO-USBNO-OUTLINE-NO-TEXT-OCTAGONAL
- R10, R9: value 10kΩ -> 0Ω
- R3, R4: value 0Ω -> 10kΩ
- renumbered IC3 to IC2
Connections:
- new net N$43: C3.2, IC1.BP
- net !CC3000_CS_3.3V: now also Q4.S, R4.1; no longer Q2.S, R6.1
- net !CC3000_CS_5V: now also J10.1, J9.1, Q4.D, R8.1; no longer J3.1, J7.1, Q2.D, R5.1
- net +3V3: now also C4.1, C6.2, IC1.OUT, R1.2, R11.2, R3.2, R4.2; no longer C4.2, R10.2, R17.2, R6.2, R8.2
- net +5V: now also C2.2, IC1.EN, IC1.IN, J7.5V, R12.2, R6.2, R8.2; no longer J4.5V, R1.2, R18.2, R9.2
- net CC3000_EN: now also J2.2; no longer J35.2
- net CC3000_IRQ_3.3V: now also Q5.S, R11.1; no longer Q4.S, R8.1
- net CC3000_IRQ_5V: now also J4.1, J5.1, Q5.D, R12.1; no longer J1.1, J2.1, Q4.D, R7.1
- net GND: now also C2.1, C3.1, C4.2, C6.1, IC1.GND, J7.GND0, J7.GND1, J7.GND2, J8.1; no longer C4.1, J378.1, J4.GND0, J4.GND1, J4.GND2
- net MISO_3.3V: now also Q1.S, R1.1; no longer Q5.S, R10.1
- net MISO_5V: now also J7.12, Q1.D, R5.1; no longer J4.12, Q5.D, R9.1
- net MOSI_3.3V: now also Q2.S, R2.1; no longer Q3.S, R17.1
- net MOSI_5V: now also J7.11_PWM, Q2.D, R6.1; no longer J4.11_PWM, Q3.D, R18.1
- net N$1: now also R10.2; no longer R3.2
- net N$103: now also C1.1; no longer C6.1
- net N$11: now also J10.2, J7.10_PWM; no longer J4.10_PWM, J7.2
- net N$15: now also R9.2; no longer R4.2
- net N$16: now also C1.2; no longer C6.2
- net N$2: now also R10.1; no longer R3.1
- net N$4: now also J5.2, J7.3_PWM; no longer J2.2, J4.3_PWM
- net N$5: now also R9.1; no longer R4.1
- net N$6: now also J7.2; no longer J1.2
- net N$7: now also J7.9_PWM, J9.2; no longer J3.2, J4.9_PWM
- net N$9: now also J7.8; no longer J4.8
- net RES_1: now also J1.2; no longer J67.2
- net RES_2: now also J1.1; no longer J67.1
- net RES_3: now also J2.1; no longer J35.1
- net SCK_3.3V: now also Q3.S, R3.1; no longer Q1.S, R2.1
- net SCK_5V: now also J7.13, Q3.D, R7.1; no longer J4.13, Q1.D, R1.1
- net WL_EN1: now also J8.3; no longer J378.3
- net WL_EN2: now also J8.2; no longer J378.2
- net WL_UART_RX: now also J3.1; no longer J37.1
- net WL_UART_TX: now also J3.2; no longer J37.2
Other:
- moved on the sheet: C4, C6, Q1, Q2, Q3, Q4, Q5, R1, R10, R2, R3, R4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

Commit message: finished silkscreen
Parts:
- removed J10, J9: SJ, freetronics-luke:SJ
- added R13: 10kΩ, freetronics-master-v1:RESISTOR0603
- added TP1, TP2, TP3: TPTP06R, testpad:TPTP06R
- C2: value 2.2µF -> 2.2pF; device freetronics-master-v1:CAP0603 -> freetronics-master-v1:CAP0402; PACKAGE 0603 -> 0402
- C3: value 470pF -> 2.2µF
- C4: value 2.2µF -> 470pF
- C5: value 2.2pF -> 2.2µF; device freetronics-master-v1:CAP0402 -> freetronics-master-v1:CAP0603; PACKAGE 0402 -> 0603
- IC1: value MIC5219-3.3YM5 -> MIC5219; ID (none) -> MIC5219-3.3YM5
- J1: value (none) -> Mode; device freetronics-master-v1:M02PTH -> freetronics-master-v1:SJ2W
- J2, J3: value (none) -> SJ; device freetronics-master-v1:M02PTH -> freetronics-luke:SJ
- J5: value SJ -> Arduino-compatible headers; device freetronics-luke:SJ -> Arduino-Various:ARDUINO-USBNO-OUTLINE-NO-TEXT-OCTAGONAL
- J7: value Arduino-compatible headers -> (none); device Arduino-Various:ARDUINO-USBNO-OUTLINE-NO-TEXT-OCTAGONAL -> freetronics-master-v1:M041.27MM
- J8: value (none) -> SJ; device freetronics-master-v1:M03PTH -> freetronics-luke:SJ
Connections:
- net !CC3000_CS_5V: now also J4.1, J8.1; no longer J10.1, J9.1
- net +3V3: now also C5.1, R12.2; no longer C4.1
- net +5V: now also C3.2, J5.5V, R13.2; no longer C2.2, J7.5V, R12.2
- net CC3000_EN: now also J7.1, R12.1; no longer J2.2
- net CC3000_IRQ_5V: now also J2.1, J3.1, R13.1; no longer J4.1, J5.1, R12.1
- net GND: now also C4.1, C5.2, J1.1, J5.GND0, J5.GND1, J5.GND2, J7.4; no longer C2.1, C4.2, J7.GND0, J7.GND1, J7.GND2, J8.1
- net MISO_5V: now also J5.12; no longer J7.12
- net MOSI_5V: now also J5.11_PWM; no longer J7.11_PWM
- net N$103: now also C2.2; no longer C5.2
- net N$104: now also C2.1; no longer C5.1
- net N$11: now also J5.10_PWM, J8.2; no longer J10.2, J7.10_PWM
- net N$4: now also J3.2, J5.3_PWM; no longer J5.2, J7.3_PWM
- net N$43: now also C4.2; no longer C3.2
- net N$6: now also J2.2, J5.2; no longer J4.2, J7.2
- net N$7: now also J5.9_PWM, J6.2; no longer J7.9_PWM, J9.2
- net N$9: now also J4.2, J5.8; no longer J6.2, J7.8
- net RES_1: now also TP1.TP; no longer J1.2
- net RES_2: now also TP2.TP; no longer J1.1
- net RES_3: now also TP3.TP; no longer J2.1
- net SCK_5V: now also J5.13; no longer J7.13
- net WL_EN1: now also J1.3; no longer J8.3
- net WL_EN2: now also J1.2; no longer J8.2
- net WL_UART_RX: now also J7.3; no longer J3.1
- net WL_UART_TX: now also J7.2; no longer J3.2
Other:
- moved on the sheet: ANT1, C1, C2, C3, C4, C5, C6, IC1, IC2, J4, J6, L1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

Commit message: changed to microstrip antenna, fixed 50Ω line
Parts:
- removed ANT1: ANT-2.45-CHP-T, SparkFun:ANTENNA2SMD5
- added A1: INVERTED_F_ANTENNA+2, antenna:INVERTED_F_ANTENNA+2
Connections:
- net GND: now also A1.GND, A1.GND@1
- net N$104: now also A1.FEED; no longer ANT1.SIGNAL
Changed lines of the file:
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@@
 <setting verticaltext="up"/>
 </settings>
-<grid distance="0.1" unitdist="inch" unit="inch" style="lines" multiple="1" display="no" altdistance="0.01" altunitdist="inch" altunit="inch"/>
+<grid distance="0.1" unitdist="inch" unit="inch" style="lines" multiple="1" display="yes" altdistance="0.01" altunitdist="inch" altunit="inch"/>
 <layers>
 <layer number="1" name="Top" color="4" fill="1" visible="no" active="no"/>
@@
 </part>
 <part name="U$61" library="freetronics-luke" deviceset="GND" device=""/>
-<part name="ANT1" library="SparkFun" deviceset="ANTENNA2" device="SMD5" value="ANT-2.45-CHP-T"/>
 <part name="J6" library="freetronics-luke" deviceset="SJ" device="" value=""/>
 <part name="J4" library="freetronics-luke" deviceset="SJ" device="" value=""/>
@@
 <attribute name="TP_SIGNAL_NAME" value=""/>
 </part>
+<part name="A1" library="antenna" deviceset="INVERTED_F_ANTENNA" device="+2"/>
+<part name="U$22" library="freetronics-luke" deviceset="GND" device=""/>
 </parts>
 <sheets>
@@
 </instance>
 <instance part="U$61" gate="G$1" x="116.84" y="86.36" rot="MR0"/>
-<instance part="ANT1" gate="G$1" x="137.16" y="116.84" smashed="yes">
-<attribute name="NAME" x="124.46" y="129.54" size="1.27" layer="95"/>
-<attribute name="VALUE" x="124.46" y="127" size="1.27" layer="96"/>
-</instance>
 <instance part="J6" gate="G$1" x="165.1" y="55.88" smashed="yes">
 <attribute name="NAME" x="164.084" y="58.928" size="1.27" layer="95"/>
@@
 <attribute name="TP_SIGNAL_NAME" x="36.83" y="128.27" size="1.778" layer="97" rot="R90"/>
 </instance>
+<instance part="A1" gate="G$1" x="147.32" y="106.68" smashed="yes"/>
+<instance part="U$22" gate="G$1" x="137.16" y="86.36" rot="MR0"/>
 </instances>
 <busses>
@@
 <pinref part="U$1" gate="G$1" pin="GND"/>
 <wire x1="101.6" y1="48.26" x2="101.6" y2="45.72" width="0.1524" layer="91"/>
+</segment>
+<segment>
+<pinref part="A1" gate="G$1" pin="GND"/>
+<wire x1="139.7" y1="104.14" x2="137.16" y2="104.14" width="0.1524" layer="91"/>
+<pinref part="U$22" gate="G$1" pin="GND"/>
+<wire x1="137.16" y1="104.14" x2="137.16" y2="101.6" width="0.1524" layer="91"/>
+<pinref part="A1" gate="G$1" pin="GND@1"/>
+<wire x1="137.16" y1="101.6" x2="137.16" y2="88.9" width="0.1524" layer="91"/>
+<wire x1="139.7" y1="101.6" x2="137.16" y2="101.6" width="0.1524" layer="91"/>
+<junction x="137.16" y="101.6"/>
 </segment>
 </net>
@@
 <pinref part="C2" gate="G$1" pin="1"/>
 <wire x1="129.54" y1="109.22" x2="127" y2="109.22" width="0.1524" layer="91"/>
+<pinref part="A1" gate="G$1" pin="FEED"/>
+<wire x1="129.54" y1="109.22" x2="139.7" y2="109.22" width="0.1524" layer="91"/>
 <junction x="129.54" y="109.22"/>
-<wire x1="137.16" y1="114.3" x2="137.16" y2="109.22" width="0.1524" layer="91"/>
-<wire x1="137.16" y1="109.22" x2="129.54" y2="109.22" width="0.1524" layer="91"/>
-<pinref part="ANT1" gate="G$1" pin="SIGNAL"/>
-</segment>
-</net>
+</segment>
+</net>
